File: Circuit/PowerUnit/PowerUnit.kicad_sch (KiCad schematic)
At the start: 155 parts, among them J1 Conn_01x02_Pin, J10 Conn_01x02_Pin, J11 Conn_01x02_Pin, J12 Conn_01x02_Pin, J13 Conn_01x02_Pin, J14 Conn_01x02_Pin, J15 Conn_01x03_Pin, J16 Conn_01x03_Pin, J17 Conn_01x03_Pin, J18 Conn_01x02_Pin, J19 Conn_01x03_Pin, J2 Conn_01x02_Pin, J20 Conn_01x02_Pin, J21 Conn_01x03_Pin, J22 Conn_01x03_Pin, J23 Conn_01x03_Pin, J24 Conn_01x03_Pin, J25 Conn_01x03_Pin, J26 Conn_01x02_Pin, J27 Conn_01x02_Pin, J28 Conn_01x02_Pin, J29 Conn_01x02_Pin, J3 Conn_01x02_Pin, J30 Conn_01x02_Pin, J31 Conn_01x02_Pin, J32 Conn_01x02_Pin, J33 Conn_01x02_Pin, J34 Conn_01x02_Pin, J35 Conn_01x02_Pin, J4 Conn_01x02_Pin, J5 Conn_01x02_Pin, J6 Conn_01x02_Pin, J7 Conn_01x02_Pin, J8 Conn_01x02_Pin, J9 Conn_01x02_Pin, K1 A31CCQ24VDC1D, K2 A31CCQ24VDC1D, K3 A31CCQ24VDC1D, Q1 2SK4017, SW1 SW_SP3T, U1 INA226, U10 YDS512F, U11 INA226, U12 M78AR05-1, U13 INA226, U14 INA226, U15 M78AR033-1, U2 YDS512F, U3 INA226, U4 NE555P, U5 YDS512F, U6 INA226, U7 YDS512F, U8 INA226, U9 NJM7812FA

Commit message: コンデンサ、ダイオード、コネクタまでフットプリント割り当て
Parts:
- removed D4, D6, D8: D_Schottky, symbol Device:D_Schottky
- removed F10, F11, F2, F3, F4, F5, F6, F7, F8, F9: 10A, symbol Device:Fuse
- removed J2, J26, J27, J28, J30, J31: Conn_01x02_Pin, symbol Connector:Conn_01x02_Pin
- added C4: 1000u, Capacitor_THT:CP_Radial_D16.0mm_P7.50mm, symbol Device:C_Polarized
- added J11, J15, J20, J25: Conn_01x02_Pin, Connector_AMASS:AMASS_XT30PW-M_1x02_P2.50mm_Horizontal, symbol Connector:Conn_01x02_Pin
- added J29: Conn_01x10_Pin, Connector_PinHeader_2.54mm:PinHeader_1x10_P2.54mm_Vertical, symbol Connector:Conn_01x10_Pin
- added J30: Conn_01x03_Pin, Connector_PinHeader_2.54mm:PinHeader_1x03_P2.54mm_Vertical, symbol Connector:Conn_01x03_Pin
- added J36, J37, J38, J39, J40: Conn_01x02_Pin, OU_Conn:Hirose_DF1EC-2P-2.5DSA_1x02_P2.5mm_Vertical, symbol Connector:Conn_01x02_Pin
- C1, C2, C37: footprint (none) -> Capacitor_SMD:C_0603_1608Metric; MPN (none) -> CC0603KRX7R9BB104
- C10: renamed from C9; footprint (none) -> Capacitor_SMD:C_0603_1608Metric; MPN (none) -> CC0603KRX7R9BB104
- C11: renamed from C12; footprint (none) -> Capacitor_THT:CP_Radial_D5.0mm_P2.00mm; MPN (none) -> ルビコンPX; MPN_URL (none) -> https://akizukidenshi.com/catalog/g/g117897/
- C12: renamed from C10; footprint (none) -> Capacitor_THT:CP_Radial_D10.0mm_P5.00mm; MPN (none) -> 100μF50V125℃ PZF; MPN_URL (none) -> https://akizukidenshi.com/catalog/g/g116871/
- C13: renamed from C11; footprint (none) -> Capacitor_THT:CP_Radial_D16.0mm_P7.50mm; MPN (none) -> ルビコンZLH; MPN_URL (none) -> https://akizukidenshi.com/catalog/g/g108442/
- C14: renamed from C13; value 4700u -> 1000u; footprint (none) -> Capacitor_THT:CP_Radial_D16.0mm_P7.50mm; MPN (none) -> ルビコンZLH; MPN_URL (none) -> https://akizukidenshi.com/catalog/g/g108442/
- C15: renamed from C14; footprint (none) -> Capacitor_THT:CP_Radial_D8.0mm_P3.50mm; MPN (none) -> 47μF63V125℃ PZJ; MPN_URL (none) -> https://akizukidenshi.com/catalog/g/g116868/
- C16: renamed from C15; footprint (none) -> Capacitor_SMD:C_0805_2012Metric; MPN (none) -> CL21A225KBQNNNE
- C17: renamed from C26; footprint (none) -> Capacitor_SMD:C_0603_1608Metric; MPN (none) -> CC0603KRX7R9BB104
- C18: renamed from C25; value 0.33u -> 0.47u; footprint (none) -> Capacitor_SMD:C_0805_2012Metric; MPN (none) -> CL21B474KBFNNNE
- C19: renamed from C16; footprint (none) -> Capacitor_SMD:C_0603_1608Metric; MPN (none) -> CC0603KRX7R9BB104
- C20: renamed from C17; footprint (none) -> Capacitor_THT:CP_Radial_D10.0mm_P5.00mm; MPN (none) -> 100μF50V125℃ PZF; MPN_URL (none) -> https://akizukidenshi.com/catalog/g/g116871/
- C21: renamed from C18; footprint (none) -> Capacitor_THT:CP_Radial_D16.0mm_P7.50mm; MPN (none) -> ルビコンZLH; MPN_URL (none) -> https://akizukidenshi.com/catalog/g/g108442/
- C22: renamed from C19; value 4700u -> 1000u; footprint (none) -> Capacitor_THT:CP_Radial_D16.0mm_P7.50mm; MPN (none) -> ルビコンZLH; MPN_URL (none) -> https://akizukidenshi.com/catalog/g/g108442/
- C23: renamed from C20; footprint (none) -> Capacitor_THT:CP_Radial_D8.0mm_P3.50mm; MPN (none) -> 47μF63V125℃ PZJ; MPN_URL (none) -> https://akizukidenshi.com/catalog/g/g116868/
- C24: renamed from C21; footprint (none) -> Capacitor_SMD:C_0805_2012Metric; MPN (none) -> CL21A225KBQNNNE
- C25: renamed from C22; footprint (none) -> Capacitor_SMD:C_0603_1608Metric; MPN (none) -> CC0603KRX7R9BB104
- C26: renamed from C23; footprint (none) -> Capacitor_THT:CP_Radial_D10.0mm_P5.00mm; MPN (none) -> 100μF50V125℃ PZF; MPN_URL (none) -> https://akizukidenshi.com/catalog/g/g116871/
- C27: renamed from C24; footprint (none) -> Capacitor_THT:CP_Radial_D16.0mm_P7.50mm; MPN (none) -> ルビコンZLH; MPN_URL (none) -> https://akizukidenshi.com/catalog/g/g108442/
- C28: renamed from C27; value 4700u -> 1000u; footprint (none) -> Capacitor_THT:CP_Radial_D16.0mm_P7.50mm; MPN (none) -> ルビコンZLH; MPN_URL (none) -> https://akizukidenshi.com/catalog/g/g108442/
- C29: renamed from C28; footprint (none) -> Capacitor_THT:CP_Radial_D8.0mm_P3.50mm; MPN (none) -> 47μF63V125℃ PZJ; MPN_URL (none) -> https://akizukidenshi.com/catalog/g/g116868/
- C3: value 4700u -> 1000u; footprint (none) -> Capacitor_THT:CP_Radial_D16.0mm_P7.50mm; MPN (none) -> ルビコンZLH; MPN_URL (none) -> https://akizukidenshi.com/catalog/g/g108442/
- C30: renamed from C29; footprint (none) -> Capacitor_SMD:C_0805_2012Metric; MPN (none) -> CL21A225KBQNNNE
- C31: renamed from C30; footprint (none) -> Capacitor_SMD:C_0603_1608Metric; MPN (none) -> CC0603KRX7R9BB104
- C32: renamed from C31; footprint (none) -> Capacitor_THT:CP_Radial_D10.0mm_P5.00mm; MPN (none) -> 100μF50V125℃ PZF; MPN_URL (none) -> https://akizukidenshi.com/catalog/g/g116871/
- C33: renamed from C32; footprint (none) -> Capacitor_THT:CP_Radial_D16.0mm_P7.50mm; MPN (none) -> ルビコンZLH; MPN_URL (none) -> https://akizukidenshi.com/catalog/g/g108442/
- C34: renamed from C33; value 4700u -> 1000u; footprint (none) -> Capacitor_THT:CP_Radial_D16.0mm_P7.50mm; MPN (none) -> ルビコンZLH; MPN_URL (none) -> https://akizukidenshi.com/catalog/g/g108442/
- C35: renamed from C34; footprint (none) -> Capacitor_SMD:C_1206_3216Metric; MPN (none) -> CL31A106KBHNNNE
- C36: renamed from C35; footprint (none) -> Capacitor_SMD:C_0603_1608Metric; MPN (none) -> CC0603KRX7R9BB104
- C38: renamed from C36; value 3.3u -> 4.7u; footprint (none) -> Capacitor_SMD:C_0805_2012Metric; MPN (none) -> CL21A475KAQNNNE
- C39: renamed from C38; value 4700u -> 1000u; footprint (none) -> Capacitor_THT:CP_Radial_D16.0mm_P7.50mm; MPN (none) -> ルビコンZLH; MPN_URL (none) -> https://akizukidenshi.com/catalog/g/g108442/
- C40: renamed from C39; footprint (none) -> Capacitor_SMD:C_1206_3216Metric; MPN (none) -> CL31A106KBHNNNE
- C41: renamed from C40; footprint (none) -> Capacitor_SMD:C_0603_1608Metric; MPN (none) -> CC0603KRX7R9BB104
- C42: renamed from C41; footprint (none) -> Capacitor_SMD:C_0603_1608Metric; MPN (none) -> CC0603KRX7R9BB104
- C43: renamed from C42; value 3.3u -> 4.7u; footprint (none) -> Capacitor_SMD:C_0805_2012Metric; MPN (none) -> CL21A475KAQNNNE
- C5: renamed from C4; value 4700u -> 1000u; footprint (none) -> Capacitor_THT:CP_Radial_D16.0mm_P7.50mm; MPN (none) -> ルビコンZLH; MPN_URL (none) -> https://akizukidenshi.com/catalog/g/g108442/
- C6: renamed from C7; footprint (none) -> Capacitor_SMD:C_0603_1608Metric; MPN (none) -> CC0603KRX7R9BB104
- C7: renamed from C5; footprint (none) -> Capacitor_THT:CP_Radial_D8.0mm_P3.50mm; MPN (none) -> 47μF63V125℃ PZJ; MPN_URL (none) -> https://akizukidenshi.com/catalog/g/g116868/
- C8: renamed from C6; footprint (none) -> Capacitor_SMD:C_0805_2012Metric; MPN (none) -> CL21A225KBQNNNE
- C9: renamed from C8; footprint (none) -> Capacitor_SMD:C_0603_1608Metric; MPN (none) -> CC0603KRX7R9BB104
- D1: footprint (none) -> LED_THT:LED_D5.0mm
- D10: renamed from D13; footprint (none) -> LED_THT:LED_D5.0mm
- D2: renamed from D3; footprint (none) -> LED_THT:LED_D5.0mm
- D3: renamed from D2; value D_TVS_Uni -> SMCJ24A; footprint (none) -> OU_Diode:SMCJSeries_LTF
- D4: renamed from D5; value D_Schottky -> SS56C; footprint (none) -> OU_Diode:DIODE_SS56C-HF_CIP
- D5: renamed from D7; footprint (none) -> LED_THT:LED_D5.0mm
- D6: renamed from D9; value D_Schottky -> SS56C; footprint (none) -> OU_Diode:DIODE_SS56C-HF_CIP
- D7: renamed from D10; value D_Schottky -> SS56C; footprint (none) -> OU_Diode:DIODE_SS56C-HF_CIP
- D8: renamed from D11; footprint (none) -> LED_THT:LED_D5.0mm
- D9: renamed from D12; value D_Schottky -> SS56C; footprint (none) -> OU_Diode:DIODE_SS56C-HF_CIP
- F1: footprint (none) -> OU_Fuse:3557-15_KEY; MPN (none) -> 3557-15, 0891030.NXS; MPN_URL (none) -> https://akizukidenshi.com/catalog/g/g118223/, https://akizu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
- J1: footprint (none) -> Connector_AMASS:AMASS_XT60PW-M_1x02_P7.20mm_Horizontal
- J10, J3, J32, J33, J34, J4, J5, J6, J7, J8, J9: footprint (none) -> Connector_AMASS:AMASS_XT30PW-M_1x02_P2.50mm_Horizontal
- J12, J13, J14, J35: footprint (none) -> OU_Conn:Hirose_DF1EC-2P-2.5DSA_1x02_P2.5mm_Vertical
- J16: renamed from J15; footprint (none) -> Connector_PinHeader_2.54mm:PinHeader_1x03_P2.54mm_Vertical
- J17: renamed from J16; footprint (none) -> Connector_PinHeader_2.54mm:PinHeader_1x03_P2.54mm_Vertical
- J18: renamed from J17; footprint (none) -> Connector_PinHeader_2.54mm:PinHeader_1x03_P2.54mm_Vertical
- J19: renamed from J18; footprint (none) -> OU_Conn:Hirose_DF1EC-2P-2.5DSA_1x02_P2.5mm_Vertical
- J2: renamed from J11; footprint (none) -> Connector_AMASS:AMASS_XT30PW-M_1x02_P2.50mm_Horizontal
- J21: renamed from J19; footprint (none) -> Connector_PinHeader_2.54mm:PinHeader_1x03_P2.54mm_Vertical
- J22: renamed from J21; footprint (none) -> Connector_PinHeader_2.54mm:PinHeader_1x03_P2.54mm_Vertical
- J23: renamed from J20; footprint (none) -> OU_Conn:Hirose_DF1EC-2P-2.5DSA_1x02_P2.5mm_Vertical
- J24: renamed from J22; footprint (none) -> Connector_PinHeader_2.54mm:PinHeader_1x03_P2.54mm_Vertical
- J26: renamed from J23; footprint (none) -> Connector_PinHeader_2.54mm:PinHeader_1x03_P2.54mm_Vertical
- J27: renamed from J24; footprint (none) -> Connector_PinHeader_2.54mm:PinHeader_1x03_P2.54mm_Vertical
- J28: renamed from J25; footprint (none) -> Connector_PinHeader_2.54mm:PinHeader_1x03_P2.54mm_Vertical
- J31: renamed from J29; footprint (none) -> OU_Conn:Hirose_DF1EC-2P-2.5DSA_1x02_P2.5mm_Vertical
- renumbered R11 to R10, R12 to R11, R13 to R12, R14 to R13, R9 to R14, R16 to R15, R17 to R16, R18 to R17, R21 to R18, R22 to R19, R19 to R20, R20 to R21, R23 to R22, R15 to R23, R10 to R9, U13 to U12, U12 to U13, U4 to U3, U3 to U4, U9 to U5, U5 to U6, U6 to U7, U7 to U8, U8 to U9
Connections:
- net +24V_CTRL: now also J19.2 (Pin_2); no longer J19.1 (Pin_1)
- net +24V_DRV: now also C14.1, C15.1, C16.1, C22.1, C23.1, C24.1, C5.1, C7.1, C8.1, J10.2 (Pin_2), J2.2 (Pin_2), J3.2 (Pin_2), J4.2 (Pin_2), J5.2 (Pin_2), J6.2 (Pin_2), J7.2 (Pin_2), J8.2 (Pin_2), J9.2 (Pin_2), U2.1 (Vin), U2.2 (Vin), U6.1 (Vin), U6.2 (Vin), U8.1 (Vin), U8.2 (Vin), C4.1, J11.2 (Pin_2)
- net +3.3V: now also J30.3 (Pin_3), J38.2 (Pin_2), J39.2 (Pin_2), J40.2 (Pin_2); no longer J33.1 (Pin_1), J34.1 (Pin_1), J35.1 (Pin_1)
- net +5V: now also J35.2 (Pin_2), J30.2 (Pin_2), J36.2 (Pin_2), J37.2 (Pin_2); no longer J32.1 (Pin_1)
- net GND: now also J12.1 (Pin_1), J14.1 (Pin_1), J19.1 (Pin_1), J31.1 (Pin_1), J32.1 (Pin_1), J33.1 (Pin_1), J34.1 (Pin_1), J35.1 (Pin_1), J29.1 (Pin_1), J30.1 (Pin_1), J36.1 (Pin_1), J37.1 (Pin_1), J38.1 (Pin_1), J39.1 (Pin_1), J40.1 (Pin_1); no longer J12.2 (Pin_2), J14.2 (Pin_2), J19.2 (Pin_2), J31.2 (Pin_2), J32.2 (Pin_2), J33.2 (Pin_2), J34.2 (Pin_2), J35.2 (Pin_2)
- net GNDPWR: now also J1.1 (Pin_1), J10.1 (Pin_1), J2.1 (Pin_1), J3.1 (Pin_1), J4.1 (Pin_1), J5.1 (Pin_1), J6.1 (Pin_1), J7.1 (Pin_1), J8.1 (Pin_1), J9.1 (Pin_1), C4.2, J11.1 (Pin_1), J15.1 (Pin_1), J20.1 (Pin_1), J25.1 (Pin_1); no longer J1.2 (Pin_2), J10.2 (Pin_2), J2.2 (Pin_2), J3.2 (Pin_2), J4.2 (Pin_2), J5.2 (Pin_2), J6.2 (Pin_2), J7.2 (Pin_2), J8.2 (Pin_2), J9.2 (Pin_2)
- net サーボ_通信8: now reaches J27.1 (Pin_1)
- net サーボ_通信8: now also J29.9 (Pin_9)
- net at J26.2 (Pin_2), J27.2 (Pin_2), J28.2 (Pin_2)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: now also J25.2 (Pin_2)
- net サーボ_通信2: now reaches J17.1 (Pin_1)
- net サーボ_通信2: now also J29.3 (Pin_3)
- net at J16.2 (Pin_2), J17.2 (Pin_2), J18.2 (Pin_2)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: now also J15.2 (Pin_2)
- net at J13.1 (Pin_1), K1.87, R4.1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: now also J12.2 (Pin_2); no longer J12.1 (Pin_1)
- net at R26.4, U11.8 (Vbus): now also J31.2 (Pin_2), J32.2 (Pin_2), J33.2 (Pin_2), J34.2 (Pin_2); no longer J31.1 (Pin_1)
- net サーボ_通信1: now reaches J16.1 (Pin_1)
- net サーボ_通信1: now also J29.2 (Pin_2)
- net サーボ_通信6: now reaches J24.1 (Pin_1)
- net サーボ_通信6: now also J29.7 (Pin_7)
- net at J21.2 (Pin_2), J22.2 (Pin_2), J24.2 (Pin_2)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: now also J20.2 (Pin_2)
- net at F1.1: now also J1.2 (Pin_2); no longer J1.1 (Pin_1)
- net サーボ_通信3: now reaches J18.1 (Pin_1)
- net サーボ_通信3: now also J29.4 (Pin_4)
- net at SW1.3: now also J14.2 (Pin_2); no longer J14.1 (Pin_1)
- net サーボ_通信4: now reaches J21.1 (Pin_1)
- net サーボ_通信4: now also J29.5 (Pin_5)
- net サーボ_通信9: now reaches J28.1 (Pin_1)
- net サーボ_通信9: now also J29.10 (Pin_10)
- net サーボ_通信7: now reaches J26.1 (Pin_1)
- net サーボ_通信7: now also J29.8 (Pin_8)
- net サーボ_通信5: now reaches J22.1 (Pin_1)
- net サーボ_通信5: now also J29.6 (Pin_6)
Other:
- note added: "サーボ汎用1"
- note added: "サーボ汎用2"
- note added: "サーボ汎用3"
- moved on the sheet: C1, C10, C11, C12, C13, C14, C15, C16, C17, C18, C19, C2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
