File: Circuit/PowerUnit/PowerUnit.kicad_sch (KiCad schematic)
At the start: 149 parts, among them J1 Conn_01x02_Pin, J10 Conn_01x02_Pin, J11 Conn_01x02_Pin, J12 Conn_01x02_Pin, J13 Conn_01x02_Pin, J14 Conn_01x02_Pin, J15 Conn_01x02_Pin, J16 Conn_01x03_Pin, J17 Conn_01x03_Pin, J18 Conn_01x03_Pin, J19 Conn_01x02_Pin, J2 Conn_01x02_Pin, J20 Conn_01x02_Pin, J21 Conn_01x03_Pin, J22 Conn_01x02_Pin, J23 Conn_01x03_Pin, J24 Conn_01x03_Pin, J25 Conn_01x02_Pin, J26 Conn_01x03_Pin, J27 Conn_01x03_Pin, J28 Conn_01x03_Pin, J29 Conn_01x10_Pin, J3 Conn_01x02_Pin, J30 Conn_01x03_Pin, J31 Conn_01x02_Pin, J32 Conn_01x02_Pin, J33 Conn_01x02_Pin, J34 Conn_01x02_Pin, J35 Conn_01x02_Pin, J36 Conn_01x02_Pin, J37 Conn_01x02_Pin, J38 Conn_01x02_Pin, J39 Conn_01x02_Pin, J4 Conn_01x02_Pin, J40 Conn_01x02_Pin, J5 Conn_01x02_Pin, J6 Conn_01x02_Pin, J7 Conn_01x02_Pin, J8 Conn_01x02_Pin, J9 Conn_01x02_Pin, K1 A31CCQ24VDC1D, K2 A31CCQ24VDC1D, K3 A31CCQ24VDC1D, Q1 2SK4017, SW2 SW_Toggle_DPDT, U1 INA226, U10 YDS512F, U11 INA226, U12 INA226, U13 M78AR05-1, U14 INA226, U15 M78AR033-1, U2 YDS512F, U3 NE555P, U4 INA226, U5 NJM7812FA, U6 YDS512F, U7 INA226, U8 YDS512F, U9 INA226

Commit message: フットプリントの割り当て完了
Parts:
- SW2: footprint (none) -> OU_Switch:1MD6-T1-B1-M1-Q-N-S
- U10, U2, U6, U8: footprint (none) -> OU_Power:YDS512F
- U13: footprint (none) -> OU_Power:M78AR05-1
- U15: footprint (none) -> OU_Power:M78AR033-1
- U5: footprint (none) -> OU_Power:NJM7812FA
Changed lines of the file:
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@@
 			)
 		)
-		(property "Footprint" ""
+		(property "Footprint" "OU_Power:M78AR033-1"
 			(at 528.32 213.995 0)
 			(hide yes)
@@
 			)
 		)
-		(property "Footprint" ""
+		(property "Footprint" "OU_Switch:1MD6-T1-B1-M1-Q-N-S"
 			(at 104.14 166.37 0)
 			(hide yes)
@@
 			)
 		)
-		(property "Footprint" ""
+		(property "Footprint" "OU_Power:YDS512F"
 			(at 279.4 234.95 0)
 			(hide yes)
@@
 			)
 		)
-		(property "Footprint" ""
+		(property "Footprint" "OU_Power:M78AR05-1"
 			(at 458.47 213.995 0)
 			(hide yes)
@@
 			)
 		)
-		(property "Footprint" ""
+		(property "Footprint" "OU_Power:YDS512F"
 			(at 121.92 234.95 0)
 			(hide yes)
@@
 			)
 		)
-		(property "Footprint" ""
+		(property "Footprint" "OU_Power:YDS512F"
 			(at 200.66 234.95 0)
 			(hide yes)
@@
 			)
 		)
-		(property "Footprint" ""
+		(property "Footprint" "OU_Power:NJM7812FA"
 			(at 201.295 58.42 0)
 			(hide yes)
@@
 			)
 		)
-		(property "Footprint" ""
+		(property "Footprint" "OU_Power:YDS512F"
 			(at 382.27 217.17 0)
 			(hide yes)

Commit message: 電流センサにフィルターを追加
Parts:
- removed D4: SS56C, OU_Diode:DIODE_SS56C-HF_CIP, symbol Device:D_Schottky
- added C12, C22, C29, C36, C44, C5, C50: 0.1u, Capacitor_SMD:C_0603_1608Metric, symbol Device:C
- added D4: 1N4148, Diode_THT:D_DO-35_SOD27_P7.62mm_Horizontal, symbol Diode:1N4148
- added R14, R15, R20, R21, R27, R28, R34, R35, R37, R38, R4, R41, R42, R6: 10, Resistor_SMD:R_0603_1608Metric, symbol Device:R
- renumbered C9 to C10, C10 to C11, C11 to C13, C12 to C14, C13 to C15, C14 to C16, C15 to C17, C16 to C18, C17 to C19, C19 to C20, C18 to C21, C20 to C23, C21 to C24, C22 to C25, C23 to C26, C24 to C27, C25 to C28, C28 to C30, C26 to C31, C29 to C32, C27 to C33, C30 to C34, C31 to C35, C32 to C37, C33 to C38, C34 to C39, C35 to C40, C36 to C41, C37 to C42, C38 to C43, C39 to C45, C40 to C46, C41 to C47, C42 to C48, C43 to C49, C5 to C6, C6 to C7, C7 to C8, C8 to C9, D3 to D2, D2 to D3, J31 to J29, J32 to J30, J33 to J31, J34 to J32, J29 to J33, J30 to J34, R2 to R1, R8 to R10, R9 to R11, R10 to R12, R11 to R13, R12 to R16, R13 to R17, R14 to R18, R15 to R19, R1 to R2, R16 to R22, R17 to R23, R23 to R24, R18 to R25, R19 to R26, R22 to R29, R24 to R30, R25 to R31, R20 to R32, R21 to R33, R26 to R36, R27 to R39, R28 to R40, R29 to R43, R30 to R44, R4 to R5, R5 to R7, R6 to R8, R7 to R9, SW2 to SW1, U4 to U3, U3 to U4
Connections:
- net GND: now also RV2.2, D4.2 (A); no longer RV2.3
- net at U12.10 (Vin+): now also C44.1, R38.2; no longer R39.2
- net at U12.9 (Vin-): now also C44.2, R37.1; no longer R39.3
- net at C13.2, R13.1, U4.2 (TRIG)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: now also D4.1 (K)
- net at R36.2: now also R35.1; no longer U11.10 (Vin+)
- net at R36.3: now also R34.2; no longer U11.9 (Vin-)
- net at R5.2: now also R6.1; no longer U1.9 (Vin-)
- net at U1.10 (Vin+): now also C5.1, R4.1; no longer R5.3
- net at U7.10 (Vin+): now also C22.1, R21.2; no longer R23.2
- net at U7.9 (Vin-): now also C22.2, R20.1; no longer R23.3
- net at U9.10 (Vin+): now also C29.1, R28.2; no longer R29.2
- net at U9.9 (Vin-): now also C29.2, R27.1; no longer R29.3
- net at R17.2: now also R15.1; no longer U3.10 (Vin+)
- net at U3.9 (Vin-): now also C12.2, R14.1; no longer R17.3
- net at U14.10 (Vin+): now also C50.1, R42.2; no longer R43.2
- net at U14.9 (Vin-): now also C50.2, R41.1; no longer R43.3
- new net: R4.2, R5.3
- new net: R38.1, R39.2
- new net: R37.2, R39.3
- new net: R14.2, R17.3
- new net: C12.1, R15.2, U3.10 (Vin+)
- new net: C5.2, R6.2, U1.9 (Vin-)
- new net: R27.2, R29.3
- new net: C36.2, R34.1, U11.9 (Vin-)
- new net: R21.1, R23.2
- new net: R20.2, R23.3
- new net: R28.1, R29.2
- new net: C36.1, R35.2, U11.10 (Vin+)
- new net: R42.1, R43.2
- new net: R41.2, R43.3
Other:
- moved on the sheet: C11, C14, C15, C16, C17, C18, C20, C23, C24, C25, C26, C27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

Commit message: 間違えていたフットプリントを一部更新
Parts:
- J1: footprint Connector_AMASS:AMASS_XT60PW-M_1x02_P7.20mm_Horizontal -> OU_Conn:AMASS_XT60PW-M
- J10, J11, J15, J2, J20, J25, J3, J30, J31, J32, J4, J5, J6, J7, J8, J9: footprint Connector_AMASS:AMASS_XT30PW-M_1x02_P2.50mm_Horizontal -> OU_Conn:AMASS_XT30PW-M
Changed lines of the file:
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@@
 			)
 		)
-		(property "Footprint" "Connector_AMASS:AMASS_XT30PW-M_1x02_P2.50mm_Horizontal"
+		(property "Footprint" "OU_Conn:AMASS_XT30PW-M"
 			(at 35.56 213.36 0)
 			(hide yes)
@@
 			)
 		)
-		(property "Footprint" "Connector_AMASS:AMASS_XT30PW-M_1x02_P2.50mm_Horizontal"
+		(property "Footprint" "OU_Conn:AMASS_XT30PW-M"
 			(at 35.56 257.81 0)
 			(hide yes)
@@
 			)
 		)
-		(property "Footprint" "Connector_AMASS:AMASS_XT30PW-M_1x02_P2.50mm_Horizontal"
+		(property "Footprint" "OU_Conn:AMASS_XT30PW-M"
 			(at 35.56 240.03 0)
 			(hide yes)
@@
 			)
 		)
-		(property "Footprint" "Connector_AMASS:AMASS_XT30PW-M_1x02_P2.50mm_Horizontal"
+		(property "Footprint" "OU_Conn:AMASS_XT30PW-M"
 			(at 35.56 275.59 0)
 			(hide yes)
@@
 			)
 		)
-		(property "Footprint" "Connector_AMASS:AMASS_XT30PW-M_1x02_P2.50mm_Horizontal"
+		(property "Footprint" "OU_Conn:AMASS_XT30PW-M"
 			(at 35.56 248.92 0)
 			(hide yes)
@@
 			)
 		)
-		(property "Footprint" "Connector_AMASS:AMASS_XT30PW-M_1x02_P2.50mm_Horizontal"
+		(property "Footprint" "OU_Conn:AMASS_XT30PW-M"
 			(at 367.03 19.05 0)
 			(hide yes)
@@
 			)
 		)
-		(property "Footprint" "Connector_AMASS:AMASS_XT60PW-M_1x02_P7.20mm_Horizontal"
+		(property "Footprint" "OU_Conn:AMASS_XT60PW-M"
 			(at 24.13 40.64 0)
 			(hide yes)
@@
 			)
 		)
-		(property "Footprint" "Connector_AMASS:AMASS_XT30PW-M_1x02_P2.50mm_Horizontal"
+		(property "Footprint" "OU_Conn:AMASS_XT30PW-M"
 			(at 35.56 231.14 0)
 			(hide yes)
@@
 			)
 		)
-		(property "Footprint" "Connector_AMASS:AMASS_XT30PW-M_1x02_P2.50mm_Horizontal"
+		(property "Footprint" "OU_Conn:AMASS_XT30PW-M"
 			(at 35.56 222.25 0)
 			(hide yes)
@@
 			)
 		)
-		(property "Footprint" "Connector_AMASS:AMASS_XT30PW-M_1x02_P2.50mm_Horizontal"
+		(property "Footprint" "OU_Conn:AMASS_XT30PW-M"
 			(at 35.56 266.7 0)
 			(hide yes)
@@
 			)
 		)
-		(property "Footprint" "Connector_AMASS:AMASS_XT30PW-M_1x02_P2.50mm_Horizontal"
+		(property "Footprint" "OU_Conn:AMASS_XT30PW-M"
 			(at 35.56 204.47 0)
 			(hide yes)
@@
 			)
 		)
-		(property "Footprint" "Connector_AMASS:AMASS_XT30PW-M_1x02_P2.50mm_Horizontal"
+		(property "Footprint" "OU_Conn:AMASS_XT30PW-M"
 			(at 196.85 162.56 0)
 			(hide yes)
@@
 			)
 		)
-		(property "Footprint" "Connector_AMASS:AMASS_XT30PW-M_1x02_P2.50mm_Horizontal"
+		(property "Footprint" "OU_Conn:AMASS_XT30PW-M"
 			(at 35.56 284.48 0)
 			(hide yes)
@@
 			)
 		)
-		(property "Footprint" "Connector_AMASS:AMASS_XT30PW-M_1x02_P2.50mm_Horizontal"
+		(property "Footprint" "OU_Conn:AMASS_XT30PW-M"
 			(at 344.17 19.05 0)
 			(hide yes)
@@
 			)
 		)
-		(property "Footprint" "Connector_AMASS:AMASS_XT30PW-M_1x02_P2.50mm_Horizontal"
+		(property "Footprint" "OU_Conn:AMASS_XT30PW-M"
 			(at 118.11 162.56 0)
 			(hide yes)
@@
 			)
 		)
-		(property "Footprint" "Connector_AMASS:AMASS_XT30PW-M_1x02_P2.50mm_Horizontal"
+		(property "Footprint" "OU_Conn:AMASS_XT30PW-M"
 			(at 275.59 162.56 0)
 			(hide yes)
@@
 			)
 		)
-		(property "Footprint" "Connector_AMASS:AMASS_XT30PW-M_1x02_P2.50mm_Horizontal"
+		(property "Footprint" "OU_Conn:AMASS_XT30PW-M"
 			(at 355.6 19.05 0)
 			(hide yes)

Commit message: 駆動系はほぼほぼ配置が終わった
Parts:
- removed J19: Conn_01x02_Pin, OU_Conn:Hirose_DF1EC-2P-2.5DSA_1x02_P2.5mm_Vertical, symbol Connector:Conn_01x02_Pin
- removed U10, U2, U6, U8: YDS512F, OU_Power:YDS512F, symbol OU_Power:YDS512F
- added J16, J22, J28, J32: Conn_01x07_Socket, OU_Power:YDS512F-Unit, symbol Connector:Conn_01x07_Socket
- C15, C24, C33: value 1000u -> 470u; footprint Capacitor_THT:CP_Radial_D16.0mm_P7.50mm -> Capacitor_THT:CP_Radial_D10.0mm_P5.00mm; MPN_URL https://akizukidenshi.com/catalog/g/g108442/ -> https://akizukidenshi.com/catalog/g/g102719/
- C16, C25, C6: value 1000u -> 220u; footprint Capacitor_THT:CP_Radial_D16.0mm_P7.50mm -> Capacitor_THT:CP_Radial_D10.0mm_P5.00mm; MPN_URL https://akizukidenshi.com/catalog/g/g108442/ -> https://akizukidenshi.com/catalog/g/g117500/
- C18, C27, C9: footprint Capacitor_SMD:C_0805_2012Metric -> Capacitor_THT:C_Disc_D6.0mm_W4.4mm_P5.00mm; MPN CL21A225KBQNNNE -> (none); MPN_URL (none) -> https://akizukidenshi.com/catalog/g/g117114/
- D4: footprint Diode_THT:D_DO-35_SOD27_P7.62mm_Horizontal -> Diode_THT:D_DO-35_SOD27_P2.54mm_Vertical_CathodeUp
- J10, J11, J15, J7, J8, J9: footprint OU_Conn:AMASS_XT30PW-M -> OU_Conn:XT30U-M
- J13: footprint OU_Conn:Hirose_DF1EC-2P-2.5DSA_1x02_P2.5mm_Vertical -> OU_Conn:Hirose_DF1E-2P-2.5DS_1x02_P2.5mm_Horizontal
- J21: renamed from J20; footprint OU_Conn:AMASS_XT30PW-M -> OU_Conn:XT30U-M
- J24: renamed from J22; footprint OU_Conn:Hirose_DF1EC-2P-2.5DSA_1x02_P2.5mm_Vertical -> OU_Conn:Hirose_DF1E-2P-2.5DS_1x02_P2.5mm_Horizontal
- J27: renamed from J25; footprint OU_Conn:AMASS_XT30PW-M -> OU_Conn:XT30U-M
- R12: footprint OU_Reg:メタルクラッド抵抗 25W100Ω -> Resistor_THT:R_Axial_Power_L25.0mm_W9.0mm_P7.62mm_Vertical; MPN_URL https://akizukidenshi.com/catalog/g/g108480/ -> https://akizukidenshi.com/catalog/g/g103991/
- R22, R8: footprint OU_Reg:メタルクラッド抵抗 25W100Ω -> Resistor_THT:R_Axial_DIN0516_L15.5mm_D5.0mm_P5.08mm_Vertical; MPN_URL https://akizukidenshi.com/catalog/g/g108484/ -> https://akizukidenshi.com/catalog/g/g111019/
- renumbered J16 to J17, J17 to J18, J18 to J19, J21 to J23, J23 to J25, J24 to J26, J26 to J29, J27 to J30, J28 to J31, J29 to J33, J30 to J34, J31 to J35, J32 to J36, J33 to J37, J34 to J38, J35 to J39, J36 to J40, J37 to J41, J38 to J42, J39 to J43, J40 to J44, U14 to U10, U15 to U11, U3 to U2, U4 to U3, U5 to U4, U7 to U5, U9 to U6, U11 to U7, U12 to U8, U13 to U9
Connections:
- net +24V_DRV: now also J16.1 (Pin_1), J16.2 (Pin_2), J22.1 (Pin_1), J22.2 (Pin_2), J28.1 (Pin_1), J28.2 (Pin_2)
- net GND: now also J32.3 (Pin_3), J32.4 (Pin_4)
- net GNDPWR: now also J16.3 (Pin_3), J16.4 (Pin_4), J22.3 (Pin_3), J22.4 (Pin_4), J28.3 (Pin_3), J28.4 (Pin_4)
- net at RV3.2: now also J22.7 (Pin_7)
- net at RV5.2: now also J32.7 (Pin_7)
- net at C37.1, C38.1, R30.1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: now also J32.5 (Pin_5), J32.6 (Pin_6)
- net at C14.1, C15.1, R17.1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: now also J16.5 (Pin_5), J16.6 (Pin_6)
- net at C31.1, C33.1, R25.1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: now also J28.5 (Pin_5), J28.6 (Pin_6)
- net at RV4.2: now also J28.7 (Pin_7)
- net at C23.1, C24.1, R18.1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: now also J22.5 (Pin_5), J22.6 (Pin_6)
- net at C30.1, C32.1, C34.1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: now also J32.1 (Pin_1), J32.2 (Pin_2)
- net at RV1.2: now also J16.7 (Pin_7)

Commit message: スペースの問題から電流センサを減らした
Parts:
- removed C11, C12, C20, C22, C28, C29, C35, C36, C42, C44, C48, C50: 0.1u, Capacitor_SMD:C_0603_1608Metric, symbol Device:C
- removed R14, R15, R20, R21, R27, R28, R34, R35, R37, R38, R41, R42: 10, Resistor_SMD:R_0603_1608Metric, symbol Device:R
- removed R17, R23, R29, R36: 10m, OU_Reg:FRM121WFR010TM, symbol Device:R_Shunt
- removed R39, R43: 50m, OU_Reg:FRM121WFR010TM, symbol Device:R_Shunt
- removed U10, U2, U5, U6, U7, U8: INA226, Package_SO:TSSOP-10_3x3mm_P0.5mm, symbol Sensor_Energy:INA226
Connections:
- net +3.3V: now also C49.1, U11.3 (VO)
- net +5V: now also C43.1, U9.3 (VO)
- net at J27.2 (Pin_2), J29.2 (Pin_2), J30.2 (Pin_2)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: now also C31.1, C33.1, J28.5 (Pin_5), J28.6 (Pin_6), R25.1
- net at J15.2 (Pin_2), J17.2 (Pin_2), J18.2 (Pin_2)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: now also C14.1, C15.1, J16.5 (Pin_5), J16.6 (Pin_6), R9.1
- net at J21.2 (Pin_2), J23.2 (Pin_2), J25.2 (Pin_2)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: now also C23.1, C24.1, J22.5 (Pin_5), J22.6 (Pin_6), R18.1
- net at C37.1, C38.1, J32.5 (Pin_5)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: now also J33.2 (Pin_2), J34.2 (Pin_2), J35.2 (Pin_2), J36.2 (Pin_2)
- no-connect marks 10 -> 4
Other:
- note removed: "Ad: 1"
- note removed: "Ad: 2"
- note removed: "Ad: 3"
- note removed: "Ad: 6"
- note removed: "Ad: 7"
- note removed: "Ad: 8"

Commit message: 全ての配置が終わった
Parts:
- removed J17, J18, J19, J23, J25, J26, J29, J30, J31, J38: Conn_01x03_Pin, Connector_PinHeader_2.54mm:PinHeader_1x03_P2.54mm_Vertical, symbol Connector:Conn_01x03_Pin
- removed J37: Conn_01x10_Pin, Connector_PinHeader_2.54mm:PinHeader_1x10_P2.54mm_Vertical, symbol Connector:Conn_01x10_Pin
- removed J44: Conn_01x02_Pin, OU_Conn:Hirose_DF1EC-2P-2.5DSA_1x02_P2.5mm_Vertical, symbol Connector:Conn_01x02_Pin
- added J16, J20, J23: Conn_01x02_Pin, OU_Conn:XT30U-M, symbol Connector:Conn_01x02_Pin
- added J37: Conn_01x03_Pin, Connector_PinHeader_2.54mm:PinHeader_1x03_P2.54mm_Vertical, symbol Connector:Conn_01x03_Pin
- C24: renamed from C30; value 1000u -> 220u; footprint Capacitor_THT:CP_Radial_D16.0mm_P7.50mm -> Capacitor_THT:CP_Radial_D10.0mm_P5.00mm; MPN_URL https://akizukidenshi.com/catalog/g/g108442/ -> https://akizukidenshi.com/catalog/g/g117500/
- C30: renamed from C38; value 1000u -> 470u; footprint Capacitor_THT:CP_Radial_D16.0mm_P7.50mm -> Capacitor_THT:CP_Radial_D10.0mm_P5.00mm; MPN_URL https://akizukidenshi.com/catalog/g/g108442/ -> https://akizukidenshi.com/catalog/g/g102719/
- J27: renamed from J34; footprint OU_Conn:AMASS_XT30PW-M -> OU_Conn:XT30U-M
- J28: renamed from J35; footprint OU_Conn:AMASS_XT30PW-M -> OU_Conn:XT30U-M
- J29: renamed from J36; footprint OU_Conn:AMASS_XT30PW-M -> OU_Conn:XT30U-M
- SW1: MPN_URL (none) -> https://akizukidenshi.com/catalog/g/g114425/
- renumbered C13 to C11, C14 to C12, C15 to C13, C16 to C14, C17 to C15, C18 to C16, C19 to C17, C21 to C18, C23 to C19, C24 to C20, C25 to C21, C26 to C22, C27 to C23, C31 to C25, C32 to C26, C33 to C27, C34 to C28, C37 to C29, C39 to C31, C40 to C32, C41 to C33, C43 to C34, C45 to C35, C46 to C36, C47 to C37, C49 to C38, J16 to J15, J15 to J17, J22 to J18, J24 to J19, J28 to J22, J27 to J24, J32 to J25, J33 to J26, J39 to J31, J40 to J32, J41 to J33, J42 to J34, J43 to J35, R16 to R14, R18 to R15, R19 to R16, R22 to R17, R24 to R18, R25 to R19, R26 to R20, R30 to R21, R31 to R22, R32 to R23, R33 to R24, R40 to R25, R44 to R26, U3 to U2, U4 to U3, U9 to U4, U11 to U5
Connections:
- net GND: now also J37.2 (Pin_2)
- net GNDPWR: now also J16.1 (Pin_1), J20.1 (Pin_1), J23.1 (Pin_1)
- net I2C_SCL: now also J37.3 (Pin_3)
- net I2C_SDA: now also J37.1 (Pin_1)
- net at C25.1, C27.1, J22.5 (Pin_5)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: now also J23.2 (Pin_2)
- net at C12.1, C13.1, J15.5 (Pin_5)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: now also J16.2 (Pin_2)
- net at C19.1, C20.1, J18.5 (Pin_5)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: now also J20.2 (Pin_2)
Other:
- note added: "サーボ汎用1.1"
- note added: "サーボ汎用1.2"
- note added: "サーボ汎用2.1"
- note added: "サーボ汎用2.2"
- note added: "サーボ汎用3.1"
- note added: "サーボ汎用3.2"
- note removed: "3.3V電源3"
- note removed: "サーボ1"
- note removed: "サーボ2"
- note removed: "サーボ3"
- note removed: "サーボ4"
- note removed: "サーボ5"
- note removed: "サーボ6"
- note removed: "サーボ7"
- note removed: "サーボ8"
- note removed: "サーボ9"
- note removed: "サーボ汎用1"
- note removed: "サーボ汎用2"
- note removed: "サーボ汎用3"
- moved on the sheet: J17, J21, J24, J34, J35
