File: Circuit/PowerUnit/PowerUnit.kicad_pcb (KiCad board)
At the start: 2 copper layers, 200 x 140 mm, 170 parts, among them J1 Conn_01x02_Pin, J10 Conn_01x02_Pin, J11 Conn_01x02_Pin, J12 Conn_01x02_Pin, J13 Conn_01x02_Pin, J14 Conn_01x02_Pin, J15 Conn_01x02_Pin, J16 Conn_01x03_Pin, J17 Conn_01x03_Pin, J18 Conn_01x03_Pin, J19 Conn_01x02_Pin, J2 Conn_01x02_Pin, J20 Conn_01x02_Pin, J21 Conn_01x03_Pin, J22 Conn_01x02_Pin, J23 Conn_01x03_Pin, J24 Conn_01x03_Pin, J25 Conn_01x02_Pin, J26 Conn_01x03_Pin, J27 Conn_01x03_Pin, J28 Conn_01x03_Pin, J29 Conn_01x02_Pin, J3 Conn_01x02_Pin, J30 Conn_01x02_Pin, J31 Conn_01x02_Pin, J32 Conn_01x02_Pin, J33 Conn_01x10_Pin, J34 Conn_01x03_Pin, J35 Conn_01x02_Pin, J36 Conn_01x02_Pin, J37 Conn_01x02_Pin, J38 Conn_01x02_Pin, J39 Conn_01x02_Pin, J4 Conn_01x02_Pin, J40 Conn_01x02_Pin, J5 Conn_01x02_Pin, J6 Conn_01x02_Pin, J7 Conn_01x02_Pin, J8 Conn_01x02_Pin, J9 Conn_01x02_Pin, K1 A31CCQ24VDC1D, K2 A31CCQ24VDC1D, K3 A31CCQ24VDC1D, Q1 2SK4017, SW1 SW_Toggle_DPDT, U1 INA226, U10 YDS512F, U11 INA226, U12 INA226, U13 M78AR05-1, U14 INA226, U15 M78AR033-1, U2 YDS512F, U3 INA226, U4 NE555P, U5 NJM7812FA, U6 YDS512F, U7 INA226, U8 YDS512F, U9 INA226

Commit message: 途中までPCBを配置
Parts:
- added REF**: MountingHole_3.2mm_M3, MountingHole:MountingHole_3.2mm_M3, F.Cu at (213.0, 25.0)
- added REF**: MountingHole_3.2mm_M3, MountingHole:MountingHole_3.2mm_M3, F.Cu at (118.0, 110.0)
- added REF**: MountingHole_3.2mm_M3, MountingHole:MountingHole_3.2mm_M3, F.Cu at (213.0, 195.0)
- added REF**: MountingHole_3.2mm_M3, MountingHole:MountingHole_3.2mm_M3, F.Cu at (23.0, 25.0)
- added REF**: MountingHole_3.2mm_M3, MountingHole:MountingHole_3.2mm_M3, F.Cu at (128.3, 195.0)
- added REF**: MountingHole_3.2mm_M3, MountingHole:MountingHole_3.2mm_M3, F.Cu at (213.0, 93.0)
- added REF**: MountingHole_3.2mm_M3, MountingHole:MountingHole_3.2mm_M3, F.Cu at (118.0, 25.0)
- added REF**: MountingHole_3.2mm_M3, MountingHole:MountingHole_3.2mm_M3, F.Cu at (23.0, 195.0)
- moved F1 224.0 mm to (208.3, 46.0), turned to -90 degrees
- moved C24 187.8 mm to (138.2, 268.0)
- moved C33 187.8 mm to (156.3, 268.0)
- moved C45 187.8 mm to (174.3, 268.0)
- moved C6 187.8 mm to (120.2, 268.0)
- moved C15 187.8 mm to (138.2, 232.9)
- moved C25 187.8 mm to (156.3, 232.9)
- moved C3 187.8 mm to (120.2, 232.9)
- moved C38 187.8 mm to (174.3, 232.9)
- moved C16 187.8 mm to (138.2, 250.4)
- moved C30 187.8 mm to (156.3, 250.4)
- moved C39 187.8 mm to (174.3, 250.4)
- moved C4 187.8 mm to (120.2, 250.4)
- moved C14 184.8 mm to (128.0, 338.5)
- moved C18 184.8 mm to (206.8, 308.2)
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Other:
- board size 200 x 140 mm -> 200 x 180 mm
- board text added: "ここらへんはI2Cとか電圧センサ用に空けておく"
- board text added: "半分は垂直にしよ"

Commit message: 駆動系はほぼほぼ配置が終わった
Parts:
- removed the J19 at (93.5, 215.0)
- removed the REF** at (213.0, 25.0)
- removed the REF** at (118.0, 110.0)
- removed the REF** at (213.0, 195.0)
- removed the REF** at (23.0, 25.0)
- removed the REF** at (128.3, 195.0)
- removed the REF** at (213.0, 93.0)
- removed the REF** at (118.0, 25.0)
- removed the REF** at (23.0, 195.0)
- removed the U10 at (-39.6, 147.9)
- removed the U2 at (-84.5, 112.3)
- removed the U6 at (-40.1, 112.2)
- removed the U8 at (-83.8, 148.5)
- added J16: Conn_01x07_Socket, OU_Power:YDS512F-Unit, F.Cu at (154.3, 85.7)
- added J22: Conn_01x07_Socket, OU_Power:YDS512F-Unit, F.Cu at (126.4, 85.7)
- added J28: Conn_01x07_Socket, OU_Power:YDS512F-Unit, F.Cu at (98.4, 85.7)
- added J32: Conn_01x07_Socket, OU_Power:YDS512F-Unit, F.Cu at (21.0, 52.5)
- added REF**: MountingHole_3.2mm_M3, MountingHole:MountingHole_3.2mm_M3, F.Cu at (84.0, 80.0)
- added REF**: MountingHole_3.2mm_M3, MountingHole:MountingHole_3.2mm_M3, F.Cu at (213.0, 129.0)
- added REF**: 電圧メータ_秋月_超小型, OU_Power:電圧メータ_秋月_超小型, F.Cu at (179.0, 25.5)
- added REF**: MountingHole_3.2mm_M3, MountingHole:MountingHole_3.2mm_M3, F.Cu at (46.0, 129.0)
- added REF**: MountingHole_3.2mm_M3, MountingHole:MountingHole_3.2mm_M3, F.Cu at (213.0, 76.2)
- C1, C10, C19, C2, C21, C5, C7, D2, R10, R11, R13, R16, R18, R19, R25, R26, R3, R4, R5, R6, R9, U1: moved to B.Cu
- C15, C24, C33: value 1000u -> 470u; footprint Capacitor_THT:CP_Radial_D16.0mm_P7.50mm -> Capacitor_THT:CP_Radial_D10.0mm_P5.00mm
- C16, C25, C6: value 1000u -> 220u; footprint Capacitor_THT:CP_Radial_D16.0mm_P7.50mm -> Capacitor_THT:CP_Radial_D10.0mm_P5.00mm
- C18, C27, C9: footprint Capacitor_SMD:C_0805_2012Metric -> Capacitor_THT:C_Disc_D6.0mm_W4.4mm_P5.00mm
- D4: footprint Diode_THT:D_DO-35_SOD27_P7.62mm_Horizontal -> Diode_THT:D_DO-35_SOD27_P2.54mm_Vertical_CathodeUp
- J10, J11, J15, J7, J8, J9: footprint OU_Conn:AMASS_XT30PW-M -> OU_Conn:XT30U-M
- J13: footprint OU_Conn:Hirose_DF1EC-2P-2.5DSA_1x02_P2.5mm_Vertical -> OU_Conn:Hirose_DF1E-2P-2.5DS_1x02_P2.5mm_Horizontal
- J21: renamed from J20; footprint OU_Conn:AMASS_XT30PW-M -> OU_Conn:XT30U-M
- J24: renamed from J22; footprint OU_Conn:Hirose_DF1EC-2P-2.5DSA_1x02_P2.5mm_Vertical -> OU_Conn:Hirose_DF1E-2P-2.5DS_1x02_P2.5mm_Horizontal
- J27: renamed from J25; footprint OU_Conn:AMASS_XT30PW-M -> OU_Conn:XT30U-M
- R12: footprint OU_Reg:メタルクラッド抵抗 25W100Ω -> Resistor_THT:R_Axial_Power_L25.0mm_W9.0mm_P7.62mm_Vertical
- R22, R8: footprint OU_Reg:メタルクラッド抵抗 25W100Ω -> Resistor_THT:R_Axial_DIN0516_L15.5mm_D5.0mm_P5.08mm_Vertical
- moved RV4 319.2 mm to (106.7, 51.4), turned to 180 degrees
- moved J31 315.1 mm to (88.3, 38.7), turned to 90 degrees
- moved R17 309.7 mm to (258.5, 128.9)
- moved J29 307.0 mm to (99.1, 40.6)
- moved RV3 306.5 mm to (134.6, 51.4), turned to 180 degrees
- moved J30 305.2 mm to (88.3, 47.6), turned to 90 degrees
- moved R18 303.6 mm to (131.3, 53.3)
- moved J26 303.4 mm to (116.2, 38.7), turned to 90 degrees
- moved J23 297.9 mm to (127.0, 40.6)
- moved J19 297.3 mm to (144.1, 38.7), turned to 90 degrees
- moved RV1 295.9 mm to (162.6, 51.4), turned to 180 degrees
- moved J17 294.4 mm to (155.6, 40.6)
- moved J25 293.8 mm to (116.2, 47.6), turned to 90 degrees
- moved R26 293.5 mm to (110.0, 53.3)
- moved C31 292.6 mm to (93.3, 71.1), turned to 180 degrees
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- renumbered J16 to J17, J17 to J18, J18 to J19, J21 to J23, J23 to J25, J24 to J26, J26 to J29, J27 to J30, J28 to J31, J29 to J33, J30 to J34, J31 to J35, J32 to J36, J33 to J37, J34 to J38, J35 to J39, J36 to J40, J37 to J41, J38 to J42, J39 to J43, J40 to J44, U14 to U10, U15 to U11, U3 to U2, U4 to U3, U5 to U4, U7 to U5, U9 to U6, U11 to U7, U12 to U8, U13 to U9
Other:
- board size 200 x 180 mm -> 177 x 114 mm
- board text added: "BAT"
- board text added: "BAT Monitor"
- board text added: "BAT Voltage"
- board text added: "DRV"
- board text added: "Delay Trim"
- board text added: "Emergency Stop"
- board text added: "Main Switch"
- board text added: "↻5.7s ↺0.24s"
- board text removed: "ここらへんはI2Cとか電圧センサ用に空けておく"
- board text removed: "半分は垂直にしよ"

Commit message: スペースの問題から電流センサを減らした
Parts:
- removed C11, C12, C20, C22, C28, C29, C35, C36, C42, C44, C48, C50: 0.1u, Capacitor_SMD:C_0603_1608Metric
- removed R14, R15, R20, R21, R27, R28, R34, R35, R37, R38, R41, R42: 10, Resistor_SMD:R_0603_1608Metric
- removed R17, R23, R29, R36: 10m, OU_Reg:FRM121WFR010TM
- removed R39, R43: 50m, OU_Reg:FRM121WFR010TM
- removed U10, U2, U5, U6, U7, U8: INA226, Package_SO:TSSOP-10_3x3mm_P0.5mm
- added REF**: MountingHole_3.2mm_M3, MountingHole:MountingHole_3.2mm_M3, F.Cu at (59.0, 44.0)
- added REF**: MountingHole_3.2mm_M3, MountingHole:MountingHole_3.2mm_M3, F.Cu at (213.0, 25.0)
- added REF**: 電圧メータ_秋月_超小型, OU_Power:電圧メータ_秋月_超小型, F.Cu at (61.6, 104.1)
- C40, C41, C43, C46, C47, C49, D7, D9: moved to B.Cu
- moved R30 305.8 mm to (-13.9, -19.1)
- moved R31 305.8 mm to (-13.9, -16.6)
- moved RV5 305.8 mm to (30.2, -5.88)
- moved C37 305.8 mm to (-36.2, 2.54)
- moved C46 274.6 mm to (45.3, 31.8)
- moved D8 274.5 mm to (137.2, 23.5), turned to 180 degrees
- moved C40 273.6 mm to (76.8, 26.2), turned to -90 degrees
- moved D5 269.0 mm to (150.5, 23.5), turned to 180 degrees
- moved C34 253.5 mm to (22.7, 6.91)
- moved D6 253.5 mm to (-9.64, -1.91)
- moved U9 253.0 mm to (62.2, 24.8), turned to -90 degrees
- moved C41 247.8 mm to (74.3, 25.5), turned to -90 degrees
- moved C47 244.9 mm to (44.6, 34.3)
- moved U11 244.7 mm to (45.1, 45.7)
- moved J41 240.9 mm to (119.3, 24.1), turned to 180 degrees
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Connections:
- C14 pad 1: Net-(J16-Pin_5) -> Net-(J15-Pin_2)
- C15 pad 1: Net-(J16-Pin_5) -> Net-(J15-Pin_2)
- C23 pad 1: Net-(J22-Pin_5) -> Net-(J21-Pin_2)
- C24 pad 1: Net-(J22-Pin_5) -> Net-(J21-Pin_2)
- C31 pad 1: Net-(J28-Pin_5) -> Net-(J27-Pin_2)
- C33 pad 1: Net-(J28-Pin_5) -> Net-(J27-Pin_2)
- C43 pad 1: Net-(U9-VO) -> +5V
- C49 pad 1: Net-(U11-VO) -> +3.3V
- J16 pad 5: Net-(J16-Pin_5) -> Net-(J15-Pin_2)
- J16 pad 6: Net-(J16-Pin_5) -> Net-(J15-Pin_2)
- J22 pad 5: Net-(J22-Pin_5) -> Net-(J21-Pin_2)
- J22 pad 6: Net-(J22-Pin_5) -> Net-(J21-Pin_2)
- J28 pad 5: Net-(J28-Pin_5) -> Net-(J27-Pin_2)
- J28 pad 6: Net-(J28-Pin_5) -> Net-(J27-Pin_2)
- J33 pad 2: Net-(J33-Pin_2) -> Net-(J32-Pin_5)
- J34 pad 2: Net-(J33-Pin_2) -> Net-(J32-Pin_5)
- J35 pad 2: Net-(J33-Pin_2) -> Net-(J32-Pin_5)
- J36 pad 2: Net-(J33-Pin_2) -> Net-(J32-Pin_5)
- R18 pad 1: Net-(J22-Pin_5) -> Net-(J21-Pin_2)
- R25 pad 1: Net-(J28-Pin_5) -> Net-(J27-Pin_2)
- R9 pad 1: Net-(J16-Pin_5) -> Net-(J15-Pin_2)
- U11 pad 3: Net-(U11-VO) -> +3.3V
- U9 pad 3: Net-(U9-VO) -> +5V

Commit message: 全ての配置が終わった
Parts:
- removed the J17 at (155.6, 40.6)
- removed the J18 at (144.1, 47.6)
- removed the J19 at (144.1, 38.7)
- removed the J25 at (116.2, 47.6)
- removed the J26 at (116.2, 38.7)
- removed the J29 at (99.1, 40.6)
- removed J30, J38: Conn_01x03_Pin, Connector_PinHeader_2.54mm:PinHeader_1x03_P2.54mm_Vertical
- removed the J31 at (88.3, 38.7)
- removed J44: Conn_01x02_Pin, OU_Conn:Hirose_DF1EC-2P-2.5DSA_1x02_P2.5mm_Vertical
- removed the REF** at (84.0, 80.0)
- added J16: Conn_01x02_Pin, OU_Conn:XT30U-M, F.Cu at (145.4, 40.1)
- added J20: Conn_01x02_Pin, OU_Conn:XT30U-M, F.Cu at (117.5, 40.1)
- added REF**: 電圧メータ_秋月_超小型, OU_Power:電圧メータ_秋月_超小型, F.Cu at (67.9, 101.4)
- C24: renamed from C30; value 1000u -> 220u; footprint Capacitor_THT:CP_Radial_D16.0mm_P7.50mm -> Capacitor_THT:CP_Radial_D10.0mm_P5.00mm
- C28: renamed from C34; moved to B.Cu
- C30: renamed from C38; value 1000u -> 470u; footprint Capacitor_THT:CP_Radial_D16.0mm_P7.50mm -> Capacitor_THT:CP_Radial_D10.0mm_P5.00mm
- D6, R2: moved to B.Cu
- J23: value Conn_01x03_Pin -> Conn_01x02_Pin; footprint Connector_PinHeader_2.54mm:PinHeader_1x03_P2.54mm_Vertical -> OU_Conn:XT30U-M
- J27: renamed from J34; footprint OU_Conn:AMASS_XT30PW-M -> OU_Conn:XT30U-M
- J28: renamed from J35; footprint OU_Conn:AMASS_XT30PW-M -> OU_Conn:XT30U-M
- J29: renamed from J36; footprint OU_Conn:AMASS_XT30PW-M -> OU_Conn:XT30U-M
- J37: value Conn_01x10_Pin -> Conn_01x03_Pin; footprint Connector_PinHeader_2.54mm:PinHeader_1x10_P2.54mm_Vertical -> Connector_PinHeader_2.54mm:PinHeader_1x03_P2.54mm_Vertical
- R21: renamed from R30; moved to B.Cu
- R22: renamed from R31; moved to B.Cu
- R23: renamed from R32; moved to B.Cu
- R24: renamed from R33; moved to B.Cu
- moved R23 279.8 mm to (156.7, 24.1), turned to 180 degrees
- moved R24 255.4 mm to (151.6, 24.1), turned to 180 degrees
- moved D10 228.5 mm to (43.2, 83.8)
- moved J37 217.9 mm to (152.4, 22.2), turned to 90 degrees
- moved R2 198.2 mm to (169.5, 36.2), turned to 180 degrees
- moved J27 181.5 mm to (54.7, 71.1)
- moved R26 181.2 mm to (43.2, 78.7)
- moved J28 164.5 mm to (54.7, 82.5)
- moved J26 154.5 mm to (45.1, 101.6), turned to -90 degrees
- moved C29 149.9 mm to (71.6, 106.7), turned to 180 degrees
- moved J29 147.1 mm to (46.4, 92.1)
- moved R21 144.2 mm to (86.1, 84.8), turned to 180 degrees
- moved R22 137.4 mm to (85.6, 78.2), turned to 180 degrees
- moved J25 131.2 mm to (79.0, 73.0), turned to 20 degrees
- moved C30 109.6 mm to (66.0, 97.2), turned to 180 degrees
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- renumbered C13 to C11, C14 to C12, C15 to C13, C16 to C14, C17 to C15, C18 to C16, C19 to C17, C21 to C18, C23 to C19, C24 to C20, C25 to C21, C26 to C22, C27 to C23, C31 to C25, C32 to C26, C33 to C27, C37 to C29, C39 to C31, C40 to C32, C41 to C33, C43 to C34, C45 to C35, C46 to C36, C47 to C37, C49 to C38, J16 to J15, J15 to J17, J22 to J18, J24 to J19, J28 to J22, J27 to J24, J32 to J25, J33 to J26, J39 to J31, J40 to J32, J41 to J33, J42 to J34, J43 to J35, R16 to R14, R18 to R15, R19 to R16, R22 to R17, R24 to R18, R25 to R19, R26 to R20, R40 to R25, R44 to R26, U3 to U2, U4 to U3, U9 to U4, U11 to U5
Connections:
- C19 pad 1: Net-(J21-Pin_2) -> Net-(J18-Pin_5)
- C20 pad 1: Net-(J21-Pin_2) -> Net-(J18-Pin_5)
- C25 pad 1: Net-(J27-Pin_2) -> Net-(J22-Pin_5)
- C27 pad 1: Net-(J27-Pin_2) -> Net-(J22-Pin_5)
- J18 pad 5: Net-(J21-Pin_2) -> Net-(J18-Pin_5)
- J18 pad 6: Net-(J21-Pin_2) -> Net-(J18-Pin_5)
- J21 pad 2: Net-(J21-Pin_2) -> Net-(J18-Pin_5)
- J22 pad 5: Net-(J27-Pin_2) -> Net-(J22-Pin_5)
- J22 pad 6: Net-(J27-Pin_2) -> Net-(J22-Pin_5)
- J23 pad 1: /サーボ_通信4 -> GNDPWR
- J23 pad 2: Net-(J21-Pin_2) -> Net-(J22-Pin_5)
- J24 pad 2: Net-(J27-Pin_2) -> Net-(J22-Pin_5)
- J37 pad 1: GND -> /I2C_SDA
- J37 pad 2: /サーボ_通信1 -> GND
- J37 pad 3: /サーボ_通信2 -> /I2C_SCL
- R15 pad 1: Net-(J21-Pin_2) -> Net-(J18-Pin_5)
- R19 pad 1: Net-(J27-Pin_2) -> Net-(J22-Pin_5)
- SW1 pad 4: Net-(J21-Pin_2) -> Net-(J18-Pin_5)
- SW1 pad 6: Net-(J27-Pin_2) -> Net-(J22-Pin_5)
Other:
- board text added: "+3.3V"
- board text added: "+5V"
- board text added: "+5V PS"
- board text added: "CTRL"
- board text added: "Current Sensor"
- board text added: "Fuse"
- board text added: "General"
- board text added: "General Voltage"
- board text added: "Meas. Selector"
- board text added: "MotorPS"
- board text added: "S1"
- board text added: "S1 S2 S3"
- board text added: "S2"
- board text added: "S3"
- board text added: "Servo Voltage"
- board text added: "ServoPS"
- board text added: "Trim General"
- board text added: "↑"
- board text added: "↓"
- board text added: "こ こ を 通 す"
