File: Circuit/PowerUnit (コピー)/_restore_backup_2026-06-16T19-05-55-319/PowerUnit.kicad_sch (KiCad schematic)
At the start: 149 parts, among them J1 Conn_01x02_Pin, J10 Conn_01x02_Pin, J11 Conn_01x02_Pin, J12 Conn_01x02_Pin, J13 Conn_01x02_Pin, J14 Conn_01x02_Pin, J15 Conn_01x02_Pin, J16 Conn_01x03_Pin, J17 Conn_01x03_Pin, J18 Conn_01x03_Pin, J19 Conn_01x02_Pin, J2 Conn_01x02_Pin, J20 Conn_01x02_Pin, J21 Conn_01x03_Pin, J22 Conn_01x02_Pin, J23 Conn_01x03_Pin, J24 Conn_01x03_Pin, J25 Conn_01x02_Pin, J26 Conn_01x03_Pin, J27 Conn_01x03_Pin, J28 Conn_01x03_Pin, J29 Conn_01x10_Pin, J3 Conn_01x02_Pin, J30 Conn_01x03_Pin, J31 Conn_01x02_Pin, J32 Conn_01x02_Pin, J33 Conn_01x02_Pin, J34 Conn_01x02_Pin, J35 Conn_01x02_Pin, J36 Conn_01x02_Pin, J37 Conn_01x02_Pin, J38 Conn_01x02_Pin, J39 Conn_01x02_Pin, J4 Conn_01x02_Pin, J40 Conn_01x02_Pin, J5 Conn_01x02_Pin, J6 Conn_01x02_Pin, J7 Conn_01x02_Pin, J8 Conn_01x02_Pin, J9 Conn_01x02_Pin, K1 A31CCQ24VDC1D, K2 A31CCQ24VDC1D, K3 A31CCQ24VDC1D, Q1 2SK4017, SW2 SW_Toggle_DPDT, U1 INA226, U10 YDS512F, U11 INA226, U12 INA226, U13 M78AR05-1, U14 INA226, U15 M78AR033-1, U2 YDS512F, U3 NE555P, U4 INA226, U5 NJM7812FA, U6 YDS512F, U7 INA226, U8 YDS512F, U9 INA226

Commit message: 一旦、切り替えスイッチまでフットプリント割り当て済み
Parts:
- removed RV2: 500k, OU_Reg:TRIM_3362P-1-103, symbol Device:R_Potentiometer_Trim
- removed SW2: SW_Toggle_DPDT, symbol Switch:SW_Push_DPDT
- added R12: 500k, symbol Device:R_Trim
- added SW1: SW_SP3T, symbol Switch:SW_SP3T
- RV1: value 20k -> 15k; footprint OU_Reg:TRIM_3296W-1-250 -> (none); MPN_URL https://akizukidenshi.com/catalog/g/g101032/ -> (none)
- RV2: renamed from RV3; value 20k -> 15k; footprint OU_Reg:TRIM_3296W-1-250 -> (none); MPN_URL https://akizukidenshi.com/catalog/g/g101032/ -> (none)
- RV3: renamed from RV4; value 20k -> 15k; footprint OU_Reg:TRIM_3296W-1-250 -> (none); MPN_URL https://akizukidenshi.com/catalog/g/g101032/ -> (none)
- RV4: renamed from RV5; value 20k -> 15k; footprint OU_Reg:TRIM_3296W-1-250 -> (none); MPN_URL https://akizukidenshi.com/catalog/g/g101032/ -> (none)
- renumbered R12 to R13, R13 to R14, R14 to R15, R15 to R16, R16 to R17, R17 to R18, R18 to R19, R19 to R20, R20 to R21, R21 to R22, R22 to R23, R23 to R24, R24 to R25, R25 to R26, R26 to R27, R27 to R28, R28 to R29, R29 to R30, R30 to R31
Connections:
- net GND: now also R12.2
- net at J25.2 (Pin_2), J26.2 (Pin_2), J27.2 (Pin_2)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: now also SW1.4
- net at J15.2 (Pin_2), J16.2 (Pin_2), J17.2 (Pin_2)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: now also SW1.1
- net at J14.2 (Pin_2): now also SW1.3
- net at J20.2 (Pin_2), J21.2 (Pin_2), J23.2 (Pin_2)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: now also SW1.2
- net at R11.2: now also R12.1
- no-connect marks 10 -> 9
Other:
- moved on the sheet: C3, C4, D1, D3, J10, J11, J2, J3, J4, J5, J6, J7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
