File: Circuit/PowerUnit_Servo/PowerUnit_Servo.kicad_pcb (KiCad board)
At the start: 2 copper layers, 100 x 60 mm, 29 parts, among them J1 Conn_01x02_Pin, J10 Conn_01x02_Pin, J11 Conn_01x02_Pin, J2 Conn_01x02_Pin, J3 Conn_01x07_Socket, J4 Conn_01x02_Pin, J5 Conn_01x02_Pin, J6 Conn_01x07_Socket, J7 Conn_01x02_Pin, J8 Conn_01x02_Pin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

Commit message: 制御電源基板が完成
Parts:
- added C1: 1u, Capacitor_THT:C_Disc_D6.0mm_W4.4mm_P5.00mm, F.Cu at (92.5, 37.0)
- added C2: 470u, Capacitor_THT:CP_Radial_D10.0mm_P5.00mm, F.Cu at (112.5, 46.0)
Routing:
- net GNDPWR: vias 65 -> 77

Commit message: 再度修正
Changed lines of the file:
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@@
+	)
+	(gr_line
+		(start 30.48 20.32)
+		(end 30.48 22.225)
+		(stroke
+			(width 0.3)
+			(type default)
+		)
+		(layer "F.SilkS")
+	)
+	(gr_line
+		(start 30.48 64.135)
+		(end 30.48 62.23)
+		(stroke
+			(width 0.3)
+			(type default)
+		)
+		(layer "F.SilkS")
+	)
+	(gr_line
+		(start 32.385 20.32)
+		(end 30.48 20.32)
+		(stroke
+			(width 0.3)
+			(type default)
+		)
+		(layer "F.SilkS")
+	)
+	(gr_line
+		(start 32.385 64.135)
+		(end 30.48 64.135)
+		(stroke
+			(width 0.3)
+			(type default)
+		)
+		(layer "F.SilkS")
 	)
 	(gr_line
@@
 	)
 	(gr_line
+		(start 53.975 20.32)
+		(end 53.975 22.225)
+		(stroke
+			(width 0.3)
+			(type default)
+		)
+		(layer "F.SilkS")
+	)
+	(gr_line
+		(start 53.975 64.135)
+		(end 53.975 62.23)
+		(stroke
+			(width 0.3)
+			(type default)
+		)
+		(layer "F.SilkS")
+	)
+	(gr_line
 		(start 55.245 68.58)
 		(end 41.91 68.58)
@@
 		(start 55.245 68.58)
 		(end 55.245 80.01)
+		(stroke
+			(width 0.3)
+			(type default)
+		)
+		(layer "F.SilkS")
+	)
+	(gr_line
+		(start 55.88 20.32)
+		(end 53.975 20.32)
+		(stroke
+			(width 0.3)
+			(type default)
+		)
+		(layer "F.SilkS")
+	)
+	(gr_line
+		(start 55.88 64.135)
+		(end 53.975 64.135)
 		(stroke
 			(width 0.3)
@@
 		(stroke
 			(width 0.3)
+			(type default)
+		)
+		(layer "F.SilkS")
+	)
+	(gr_line
+		(start 78.105 20.32)
+		(end 80.01 20.32)
+		(stroke
+			(width 0.3)
+			(type default)
+		)
+		(layer "F.SilkS")
+	)
+	(gr_line
+		(start 78.105 22.225)
+		(end 78.105 20.32)
+		(stroke
+			(width 0.3)
+			(type default)
+		)
+		(layer "F.SilkS")
+	)
+	(gr_line
+		(start 78.105 62.23)
+		(end 78.105 64.135)
+		(stroke
+			(width 0.3)
+			(type default)
+		)
+		(layer "F.SilkS")
+	)
+	(gr_line
+		(start 78.105 64.135)
+		(end 79.375 64.135)
+		(stroke
+			(width 0.3)
