File: Circuit/PowerUnit_Servo/PowerUnit_Servo.kicad_sch (KiCad schematic)
At the start: 25 parts, among them J1 Conn_01x02_Pin, J10 Conn_01x02_Pin, J11 Conn_01x02_Pin, J2 Conn_01x02_Pin, J3 Conn_01x07_Socket, J4 Conn_01x02_Pin, J5 Conn_01x02_Pin, J6 Conn_01x07_Socket, J7 Conn_01x02_Pin, J8 Conn_01x02_Pin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

Commit message: 発注用データを用意 発注した
Parts:
- D1: MPN_URL (none) -> https://akizukidenshi.com/catalog/g/g111333/
- J1: MPN_URL (none) -> https://akizukidenshi.com/catalog/g/g118156/
- R1: MPN_URL (none) -> https://akizukidenshi.com/catalog/g/g125752/
- R2, R4, R6: MPN_URL (none) -> https://akizukidenshi.com/catalog/g/g116123/
- R3, R5, R7: MPN_URL (none) -> https://akizukidenshi.com/catalog/g/g125152/
Changed lines of the file:
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@@
+			)
+		)
+		(property "MPN_URL" "https://akizukidenshi.com/catalog/g/g116123/"
+			(at 179.07 77.47 0)
+			(hide yes)
+			(show_name no)
+			(do_not_autoplace no)
+			(effects
+				(font
+					(size 1.27 1.27)
+				)
 			)
 		)
@@
 			)
 		)
+		(property "MPN_URL" "https://akizukidenshi.com/catalog/g/g125152/"
+			(at 87.63 97.79 0)
+			(hide yes)
+			(show_name no)
+			(do_not_autoplace no)
+			(effects
+				(font
+					(size 1.27 1.27)
+				)
+			)
+		)
 		(pin "2"
 		)
@@
 			)
 		)
+		(property "MPN_URL" "https://akizukidenshi.com/catalog/g/g111333/"
+			(at 50.8 69.85 90)
+			(hide yes)
+			(show_name no)
+			(do_not_autoplace no)
+			(effects
+				(font
+					(size 1.27 1.27)
+				)
+			)
+		)
 		(pin "1"
 		)
@@
 			)
 		)
+		(property "MPN_URL" "https://akizukidenshi.com/catalog/g/g125152/"
+			(at 133.35 97.79 0)
+			(hide yes)
+			(show_name no)
+			(do_not_autoplace no)
+			(effects
+				(font
+					(size 1.27 1.27)
+				)
+			)
+		)
 		(pin "2"
 		)
@@
 			)
 		)
+		(property "MPN_URL" "https://akizukidenshi.com/catalog/g/g118156/"
+			(at 26.67 49.53 90)
+			(hide yes)
+			(show_name no)
+			(do_not_autoplace no)
+			(effects
+				(font
+					(size 1.27 1.27)
+				)
+			)
+		)
 		(pin "2"
 		)
@@
 			)
 		)
+		(property "MPN_URL" "https://akizukidenshi.com/catalog/g/g116123/"
+			(at 133.35 77.47 0)
+			(hide yes)
+			(show_name no)
+			(do_not_autoplace no)
+			(effects
+				(font
+					(size 1.27 1.27)
+				)
+			)
+		)
 		(pin "1"
 		)
@@
 			)
 		)
+		(property "MPN_URL" "https://akizukidenshi.com/catalog/g/g116123/"
+			(at 87.63 77.47 0)
+			(hide yes)
+			(show_name no)
+			(do_not_autoplace no)
+			(effects
+				(font
+					(size 1.27 1.27)
+				)
+			)
+		)
 		(pin "1"
 		)
@@
 			)
 		)
+		(property "MPN_URL" "https://akizukidenshi.com/catalog/g/g125152/"
+			(at 179.07 97.79 0)
+			(hide yes)
+			(show_name no)
+			(do_not_autoplace no)
+			(effects
+				(font
+					(size 1.27 1.27)
+				)
+			)
+		)
 		(pin "2"
 		)
@@
 			(at 50.8 60.96 90)
 			(hide yes)
+			(show_name no)
+			(do_not_autoplace no)
+			(effects
+				(font
+					(size 1.27 1.27)
+				)
+			)
+		)
+		(property "MPN_URL" "https://akizukidenshi.com/catalog/g/g125752/"
+			(at 50.8 60.96 90)
+			(hide yes)
