File: Circuit/PowerUnit_Control/PowerUnit_Control.kicad_pcb (KiCad board)
At the start: 2 copper layers, 100 x 47 mm, 40 parts, among them J1 Conn_01x02_Pin, J10 Conn_01x02_Pin, J11 Conn_01x02_Pin, J2 Conn_01x02_Pin, J3 Conn_01x07_Socket, J4 Conn_01x02_Pin, J5 Conn_01x02_Pin, J6 Conn_01x02_Pin, J7 Conn_01x02_Pin, J8 Conn_01x02_Pin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

Commit message: 再度修正
Parts:
- added F1: 5A, OU_Fuse:FUC-03A, F.Cu at (149.0, 23.5)
Connections:
- J1 pad 2: Net-(D2-A) -> Net-(J1-Pin_2)
Routing:
- net Net-(D2-A): track 13.9 -> 40.4 mm
- added copper zone on B.Cu, net Net-(J1-Pin_2)
